File: module-basic-ui.brd (EAGLE design)
At the start: 49.8 x 23.4 mm, 10 parts

Commit message: board labels tweak
Parts:
- moved U$4 1.78 mm to (24.6, 11.2)
Changed lines of the file:
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@@
 <attribute name="VALUE" x="47.244" y="5.715" size="1.27" layer="27" ratio="10" rot="R90"/>
 </element>
-<element name="U$4" library="SparkFun-Aesthetics" package="OSHW-LOGO-M" value="" x="24.638" y="9.398" rot="MR0"/>
+<element name="U$4" library="SparkFun-Aesthetics" package="OSHW-LOGO-M" value="" x="24.638" y="11.176" rot="MR0"/>
 <element name="JP1" library="SparkFun-Connectors" package="1X04" value="" x="15.748" y="5.588" smashed="yes" rot="R90">
 <attribute name="VALUE" x="18.923" y="4.318" size="1.27" layer="27" rot="R90"/>
